File: hardware/Main Board/Main Board.sch (KiCad schematic (older format))
At the start: 18 parts, among them J1 DEC Motor, J2 RA Motor, J3 Battery, J4 OLED Display, J6 Fan, P1 Conn_02x20_Odd_Even, Q6 S8050, U1 ELEGOO, U2 RA Driver, U3 BuckConverter, U4 BuckConverter

Commit message: Indicate the wattage of R13.
Signed-off-by: John Jacques <eruditelite@gmail.com>
Parts:
- R13: Wattage (none) -> 1/8
Changed lines of the file:
@@
 F 2 "Resistor_THT:R_Axial_DIN0204_L3.6mm_D1.6mm_P1.90mm_Vertical" V 9380 1800 50  0001 C CNN
 F 3 "~" H 9450 1800 50  0001 C CNN
+F 4 "1/8" V 9450 1800 50  0001 C CNN "Wattage"
 	1    9450 1800
 	0    1    1    0
